Commit message: Add RGB-D social navigation and people-aware planning

File: ros2_omni_robot_sim/urdf/3w_v2_multi/base_link.urdf.xacro (robot description, xacro)
@@ -4,9 +4,11 @@
   <xacro:include filename="$(find ros2_omni_robot_sim)/urdf/3w_v2_multi/omni_wheel.urdf.xacro"/>
   <xacro:include filename="$(find ros2_omni_robot_sim)/urdf/3w_v2_multi/camera.urdf.xacro"/>
+  <xacro:include filename="$(find ros2_omni_robot_sim)/urdf/3w_v2_multi/leader_camera.urdf.xacro"/>
   <xacro:include filename="$(find ros2_omni_robot_sim)/urdf/3w_v2_multi/lidar.urdf.xacro"/>
   <xacro:include filename="$(find ros2_omni_robot_sim)/urdf/3w_v2_multi/imu.urdf.xacro"/>
   <xacro:macro
       name="base_link"
-      params="parent xyz rpy prefix">
+      params="parent xyz rpy prefix leader_camera_enabled:=false camera_width:=640 camera_height:=480 camera_rate:=15.0">
+    <xacro:property name="camera_active" value="${str(leader_camera_enabled).lower() in ('true', '1')}"/>
     <!-- ==================== BASE ==================== -->
     <link name="base_link">
@@ -57,5 +59,6 @@
         rpy="-0.8040 1.5708 -2.8984"/>
     <!-- ==================== CAMERA ==================== -->
-    <xacro:camera
+    <xacro:unless value="${camera_active}">
+      <xacro:camera
         parent="base_link"
         suffix="1"
@@ -63,10 +66,16 @@
         rpy="0 0 0"
         prefix="${prefix}"/>
+    </xacro:unless>
+    <xacro:if value="${camera_active}">
+      <xacro:leader_camera parent="base_link" prefix="${prefix}"
+          width="${camera_width}" height="${camera_height}" rate="${camera_rate}"/>
+    </xacro:if>
     <!-- ==================== LIDAR ==================== -->
     <xacro:lidar
         parent="base_link"
         suffix="1"
-        xyz="0.0000 0.0000 0.1010"
+        xyz="0.0000 0.0000 ${0.330 if camera_active else 0.101}"
         rpy="0 0 0"
+        multilayer="${camera_active}"
         prefix="${prefix}"/>
     <!-- ==================== IMU ==================== -->

File: ros2_omni_robot_sim/urdf/3w_v2_multi/lidar.urdf.xacro (robot description, xacro)
@@ -1,7 +1,9 @@
 <?xml version="1.0"?>
 <robot xmlns:xacro="http://ros.org/wiki/xacro">
-  <xacro:macro name="lidar" params="suffix parent xyz rpy prefix">
+  <xacro:macro name="lidar" params="suffix parent xyz rpy prefix multilayer:=false">
+    <xacro:property name="is_multilayer" value="${str(multilayer).lower() in ('true', '1')}"/>
+    <xacro:property name="lidar_link" value="${'leader_lidar_link' if is_multilayer else prefix + '/lidar_link_' + str(suffix)}"/>
     <!-- LiDAR link -->
-    <link name="${prefix}/lidar_link_${suffix}">
+    <link name="${lidar_link}">
       <visual>
         <geometry>
@@ -20,5 +22,5 @@
       type="fixed">
       <parent link="${parent}" />
-      <child link="${prefix}/lidar_link_${suffix}" />
+      <child link="${lidar_link}" />
       <origin
         xyz="${xyz}"
@@ -27,5 +29,5 @@
     </joint>
     <!-- Gazebo LiDAR -->
-    <gazebo reference="${prefix}/lidar_link_${suffix}">
+    <gazebo reference="${lidar_link}">
       <sensor
         name="${prefix}_gpu_lidar"
@@ -34,5 +36,5 @@
         <update_rate>5</update_rate>
         <gz_frame_id>
-          ${prefix}/lidar_link_${suffix}
+          ${prefix + '/leader_lidar_link' if is_multilayer else prefix + '/lidar_link_' + str(suffix)}
         </gz_frame_id>
         <ray>
@@ -44,4 +46,14 @@
               <max_angle>3.1415</max_angle>
             </horizontal>
+            <!-- The elevated leader scans down to the floor as well as
+                 horizontally. Its point cloud is height-filtered into /scan. -->
+            <xacro:if value="${is_multilayer}">
+              <vertical>
+                <samples>91</samples>
+                <resolution>1</resolution>
+                <min_angle>${-pi/3}</min_angle>
+                <max_angle>0</max_angle>
+              </vertical>
+            </xacro:if>
           </scan>
           <range>

File: ros2_omni_robot_sim/urdf/3w_v2_multi/main.urdf.xacro (robot description, xacro)
@@ -6,4 +6,8 @@
     name="robot_prefix"
     default="robot1"/>
+  <xacro:arg name="leader_camera_enabled" default="false"/>
+  <xacro:arg name="camera_width" default="640"/>
+  <xacro:arg name="camera_height" default="480"/>
+  <xacro:arg name="camera_rate" default="15.0"/>
   <xacro:include
     filename="$(find ros2_omni_robot_sim)/urdf/3w_v2_multi/base_link.urdf.xacro"/>
@@ -17,4 +21,8 @@
     xyz="0 0 0"
     rpy="0 0 0"
-    prefix="$(arg robot_prefix)"/>
+    prefix="$(arg robot_prefix)"
+    leader_camera_enabled="$(arg leader_camera_enabled)"
+    camera_width="$(arg camera_width)"
+    camera_height="$(arg camera_height)"
+    camera_rate="$(arg camera_rate)"/>
 </robot>
